File: flashing-led.kicad_pcb (KiCad board)
At the start: 2 copper layers, 19 x 12.7 mm, 6 parts, among them U1 NE555

Commit message: updated schematic and pcb
Parts:
- added J1: USB_B_Micro, Connector_USB:USB_Micro-B_Molex_47346-0001, F.Cu at (156.7, 94.5)
- D1: footprint LED_SMD:LED-APA102-2020 -> LED_SMD:LED_0805_2012Metric
- R1: value 1k -> 100k; footprint Resistor_SMD:R_0201_0603Metric -> Resistor_SMD:R_0805_2012Metric
- R2: footprint Resistor_SMD:R_0201_0603Metric -> Resistor_SMD:R_0805_2012Metric
- R3: value 1k -> 270k; footprint Resistor_SMD:R_0201_0603Metric -> Resistor_SMD:R_0805_2012Metric
- U1: value NE555 -> NE555D; footprint Package_DIP:Fairchild_LSOP-8 -> Package_SO:SOIC-8_3.9x4.9mm_P1.27mm
- moved R1 23.9 mm to (147.3, 98.0)
- moved R2 20.3 mm to (151.3, 93.6)
- moved R3 14.9 mm to (143.5, 98.0), turned to 0 degrees
- moved D1 13.9 mm to (139.7, 98.0), turned to 0 degrees
- moved C1 13.2 mm to (139.7, 93.0), turned to 90 degrees
- moved U1 12.5 mm to (146.1, 93.6)
Connections:
- net +9V renamed +5V
Routing:
- net +5V: track 5.61 -> 21.1 mm, vias 3 -> 2
- net Net-(R3-Pad2): track 3.05 -> 7.31 mm
- net Net-(D1-Pad2): track 5.36 -> 1.94 mm
- net tr_thr: track 15.3 -> 13.8 mm, vias 2 -> 0
- net GND: track 2.49 -> 1.22 mm, vias 0 -> 43
- net dis: track 14.3 -> 14.0 mm, vias 2 -> 0
- added copper zone on B.Cu, net GND
- removed copper zone on B.Cu, net +5V
Other:
- board size 19 x 12.7 mm -> 22.9 x 12.2 mm
- board text added: "555 TIMER LED FLASH"
- board text added: "KARL NOORY 15-06-2020"
